File: pcb/REV2/PCB WLED Spec 7/PCB WLED Spec 7.kicad_pcb (KiCad board)
At the start: 2 copper layers, 30 x 20 mm, 55 parts, among them J1 USB_C_Receptacle_USB2.0_16P, Q1 BC807, U1 ESP32-C3, U2 RT9013-33GB, U3 LMR14050SDDAR, Y1 XRCGB40M000F1S1DR0

Commit message: pcb finished or I hope so
Routing:
- net GND: track 49.0 -> 52.6 mm, vias 202 -> 207
- net LED1_IN: track 32.0 -> 29.4 mm
- net BOOT: track 27.1 -> 29.3 mm
Changed lines of the file:
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@@
 	)
 	(via
-		(at 191.5 82.81)
+		(at 191.56 82.62)
 		(size 0.6)
 		(drill 0.3)
@@
 	)
 	(via
-		(at 190.83 82.12)
+		(at 190.87 81.94)
 		(size 0.6)
 		(drill 0.3)
@@
 	)
 	(via
-		(at 191.47 82.17)
+		(at 191.58 81.99)
 		(size 0.6)
 		(drill 0.3)
@@
 	)
 	(via
+		(at 194.55 89.54)
+		(size 0.6)
+		(drill 0.3)
+		(layers "F.Cu" "B.Cu")
+		(free yes)
+		(net 1)
+	)
+	(via
 		(at 188.62 77.96)
 		(size 0.6)
@@
 	)
 	(via
+		(at 195.93 89.54)
+		(size 0.6)
+		(drill 0.3)
+		(layers "F.Cu" "B.Cu")
+		(free yes)
+		(net 1)
+	)
+	(via
 		(at 205.5 88.75)
 		(size 0.6)
@@
 	)
 	(via
+		(at 195.25 89.54)
+		(size 0.6)
+		(drill 0.3)
+		(layers "F.Cu" "B.Cu")
+		(free yes)
+		(net 1)
+	)
+	(via
 		(at 207.75 79.75)
 		(size 0.6)
@@
 	)
 	(via
-		(at 190.87 82.81)
+		(at 190.84 82.6)
 		(size 0.6)
 		(drill 0.3)
@@
 	)
 	(via
+		(at 190.86 81.23)
+		(size 0.6)
+		(drill 0.3)
+		(layers "F.Cu" "B.Cu")
+		(free yes)
+		(net 1)
+	)
+	(via
 		(at 207.75 79)
 		(size 0.6)
@@
 	)
 	(via
+		(at 193.74 89.54)
+		(size 0.6)
+		(drill 0.3)
+		(layers "F.Cu" "B.Cu")
+		(free yes)
+		(net 1)
+	)
+	(via
 		(at 205.5 78.25)
 		(size 0.6)
@@
 	)
 	(segment
+		(start 196.7035 82.8965)
+		(end 197.3 82.3)
+		(width 0.157)
+		(layer "B.Cu")
+		(net 1)
+	)
+	(segment
 		(start 187.285 73.165)
 		(end 185.625 74.825)
@@
 	)
 	(segment
+		(start 194.44 82.3)
+		(end 194.44 82.609999)
+		(width 0.157)
+		(layer "B.Cu")
+		(net 1)
+	)
+	(segment
 		(start 194.75 70.59)
 		(end 194.75 71.04)
@@
 	)
 	(segment
+		(start 194.726501 82.8965)
+		(end 196.7035 82.8965)
+		(width 0.157)
+		(layer "B.Cu")
+		(net 1)
+	)
+	(segment
+		(start 194.44 82.609999)
+		(end 194.726501 82.8965)
+		(width 0.157)
+		(layer "B.Cu")
+		(net 1)
+	)
+	(segment
 		(start 191.9 70.335)
 		(end 194.495 70.335)
@@
 	)
 	(segment
-		(start 181.3 86.38)
-		(end 181.44 86.24)
+		(start 182.34 86.24)
+		(end 181.3 87.28)
 		(width 0.2)
 		(layer "F.Cu")
@@
 	)
 	(segment
-		(start 181.3 88)
-		(end 181.3 86.38)
+		(start 181.3 87.28)
+		(end 181.3 88)
 		(width 0.2)
 		(layer "F.Cu")
@@
 	)
 	(via
-		(at 181.44 86.24)
+		(at 182.34 86.24)
 		(size 0.6)
 		(drill 0.3)
@@
 	)
 	(segment
-		(start 181.73 85.95)
-		(end 181.44 86.24)
+		(start 193.61 88.59)
+		(end 196.2 88.59)
 		(width 0.25)
 		(layer "B.Cu")
@@
 	)
 	(segment
-		(start 199.68 83.826396)
-		(end 197.556396 85.95)
+		(start 182.34 86.24)
+		(end 191.26 86.24)
 		(width 0.25)
 		(layer "B.Cu")
@@
 	)
 	(segment
-		(start 197.59 80)
-		(end 199.68 82.09)
+		(start 191.26 86.24)
+		(end 193.61 88.59)
 		(width 0.25)
 		(layer "B.Cu")
@@
 	)
 	(segment
-		(start 197.556396 85.95)
-		(end 181.73 85.95)
+		(start 196.4 85.68)
+		(end 199.68 82.4)
 		(width 0.25)
 		(layer "B.Cu")
@@
 	(segment
 		(start 199.68 82.09)
-		(end 199.68 83.826396)
+		(end 197.59 80)
 		(width 0.25)
 		(layer "B.Cu")
@@
 	)
 	(segment
+		(start 196.2 88.59)
+		(end 196.4 88.39)
+		(width 0.25)
+		(layer "B.Cu")
+		(net 11)
+	)
+	(segment
+		(start 196.4 88.39)
+		(end 196.4 85.68)
+		(width 0.25)
+		(layer "B.Cu")
+		(net 11)
+	)
+	(segment
+		(start 199.68 82.4)
+		(end 199.68 82.09)
+		(width 0.25)
+		(layer "B.Cu")
+		(net 11)
+	)
+	(segment
 		(start 195.199999 75.438966)
 		(end 195.245 75.483967)
@@
 	)
 	(segment
-		(start 186.64 72.943408)
-		(end 185.128408 74.455)
+		(start 185.128408 74.455)
+		(end 184.555 74.455)
 		(width 0.25)
 		(layer "B.Cu")
@@
 	)
 	(segment
-		(start 188.87 84.65)
-		(end 197.89 84.65)
+		(start 198.07 82.8)
+		(end 198.07 81.64)
 		(width 0.25)
 		(layer "B.Cu")
@@
 	)
 	(segment
-		(start 183.69 75.568858)
-		(end 182.71 76.548858)
+		(start 182.71 76.548858)
+		(end 182.71 78.49)
 		(width 0.25)
 		(layer "B.Cu")
@@
 	)
 	(segment
-		(start 184.555 74.455)
-		(end 183.69 75.32)
+		(start 198.07 81.64)
+		(end 196.905 80.475)
 		(width 0.25)
 		(layer "B.Cu")
@@
 	)
 	(segment
-		(start 183.69 75.32)
-		(end 183.69 75.568858)
+		(start 184.555 74.455)
+		(end 183.69 75.32)
 		(width 0.25)
 		(layer "B.Cu")
@@
 	)
 	(segment
-		(start 186.64 72.14)
-		(end 186.64 72.943408)
+		(start 196.905 80.475)
+		(end 196.225 80.475)
 		(width 0.25)
 		(layer "B.Cu")
@@
 	)
 	(segment
-		(start 182.71 78.49)
-		(end 188.87 84.65)
+		(start 187.52 83.3)
+		(end 197.57 83.3)
 		(width 0.25)
 		(layer "B.Cu")
@@
 	)
 	(segment
-		(start 197.89 84.65)
-		(end 198.82 83.72)
+		(start 186.64 72.14)
+		(end 186.64 72.943408)
 		(width 0.25)
 		(layer "B.Cu")
@@
 	)
 	(segment
-		(start 196.835 80.475)
-		(end 196.225 80.475)
+		(start 183.69 75.32)
+		(end 183.69 75.568858)
 		(width 0.25)
 		(layer "B.Cu")
@@
 	)
 	(segment
-		(start 182.71 76.548858)
-		(end 182.71 78.49)
+		(start 186.64 72.943408)
+		(end 185.128408 74.455)
 		(width 0.25)
 		(layer "B.Cu")
@@
 	)
 	(segment
-		(start 198.82 83.72)
-		(end 198.82 82.46)
+		(start 183.69 75.568858)
+		(end 182.71 76.548858)
 		(width 0.25)
 		(layer "B.Cu")
@@
 	)
 	(segment
-		(start 185.128408 74.455)
-		(end 184.555 74.455)
+		(start 182.71 78.49)
+		(end 187.52 83.3)
 		(width 0.25)
 		(layer "B.Cu")
@@
 	)
 	(segment
-		(start 198.82 82.46)
-		(end 196.835 80.475)
+		(start 197.57 83.3)
+		(end 198.07 82.8)
 		(width 0.25)
 		(layer "B.Cu")
